File: kbv3.kicad_sch (KiCad schematic)
At the start: 23 parts, among them SW1 SW_Push, SW10 SW_Push, SW11 SW_Push, SW12 SW_Push, SW13 SW_Push, SW14 SW_Push, SW15 SW_Push, SW16 SW_Push, SW17 SW_Push, SW18 SW_Push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

Commit message: left and right
Parts:
- removed Trackball1: ~, Trackball:Trackball_footprint, symbol Trackball_symbol:Trackball
- SW1, SW10, SW11, SW12, SW13, SW14, SW15, SW16, SW17, SW18, SW19, SW2, SW20, SW21, SW3, SW4, SW5, SW6, SW7, SW8, SW9: footprint Kailh_socket_MX:Kailh_socket_MX -> Kailh_socket_MX:Kailh_socket_MX_footprint
Connections:
- no-connect marks 9 -> 11
